File: nRF52840-BBoard.kicad_sch (KiCad schematic)
At the start: 31 parts, among them J1 Conn_02x05_Odd_Even, J2 USB_C_Receptacle_USB2.0, J3 JST BATTERY INPUT, J4 Conn_01x20, J5 Conn_01x16, Q1 AO3407, SW1 SW_Push, U1 E73-2G4M08S1C-52840, U2 LTC4054, U3 AP2112K-3.3, Y1 32.768kHz

Commit message: small changes to schematic
Other:
- company: (none) -> ddB0515
- title: (none) -> nRF52840 BBoard
Changed lines of the file:
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@@
 (kicad_sch (version 20210406) (generator eeschema)
   (paper "A4")
+  (title_block
+    (title "nRF52840 BBoard")
+    (date "2021-06-04")
+    (rev "v2")
+    (company "ddB0515")
+    (comment 4 "License: CERN OHL v1.2")
+  )
   (junction (at 37.211 126.746) (diameter 1.016) (color 0 0 0 0))
   (junction (at 40.513 164.719) (diameter 1.016) (color 0 0 0 0))
